File: scheme/lpc-programmer/lpc-programmer.kicad_pcb (KiCad board)
At the start: 2 copper layers, 16 x 26 mm, 11 parts, among them J1 DB25, P1 mosi, P2 miso, P3 cs, P4 gnd

Commit message: a
Parts:
- moved J1 5.59 mm to (126.8, 128.8)
Routing:
- net GND: track 14.2 -> 44.2 mm, vias 0 -> 1
- net /p2: track 3.05 -> 18.9 mm
- net /p8: track 3.05 -> 11.7 mm
- net /p9: track 3.05 -> 11.2 mm
- added copper zone on B.Cu, net GND
- added copper zone on F.Cu, net GND
Other:
- board size 16 x 26 mm -> 23 x 35.8 mm
Changed lines of the file:
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@@
   (general
     (links 14)
-    (no_connects 5)
-    (area 0 0 0 0)
+    (no_connects 0)
+    (area 110.040599 99.173599 151.050001 153.326401)
     (thickness 1.6)
-    (drawings 10)
-    (tracks 28)
+    (drawings 20)
+    (tracks 49)
     (zones 0)
     (modules 11)
@@
     (pad_to_mask_clearance 0)
     (aux_axis_origin 0 0)
-    (visible_elements FFFFFFBF)
+    (visible_elements 7FFFFFFF)
     (pcbplotparams
       (layerselection 3178497)
@@
   )
   (module DB25M_CI (layer F.Cu)
-    (at 121.75 126.25 90)
+    (at 126.75 128.75 90)
     (descr "Connecteur DB25 male couche")
     (tags "CONN DB25")
@@
     )
   )
+  (gr_line (start 133 143) (end 133 143.25) (angle 90) (layer Edge.Cuts) (width 0.1))
+  (gr_line (start 135 141) (end 133 143) (angle 90) (layer Edge.Cuts) (width 0.1))
+  (gr_line (start 133 146.25) (end 133 143.25) (angle 90) (layer Edge.Cuts) (width 0.1))
+  (gr_line (start 132.5 146.75) (end 133 146.25) (angle 90) (layer Edge.Cuts) (width 0.1))
+  (gr_line (start 128 146.75) (end 132.5 146.75) (angle 90) (layer Edge.Cuts) (width 0.1))
+  (gr_line (start 128 146.25) (end 128 146.75) (angle 90) (layer Edge.Cuts) (width 0.1))
+  (gr_line (start 128 111) (end 128 146.25) (angle 90) (layer Edge.Cuts) (width 0.1))
+  (gr_line (start 132.5 111) (end 128 111) (angle 90) (layer Edge.Cuts) (width 0.1))
+  (gr_line (start 133 111.5) (end 132.5 111) (angle 90) (layer Edge.Cuts) (width 0.1))
+  (gr_line (start 133 113) (end 133 111.5) (angle 90) (layer Edge.Cuts) (width 0.1))
+  (gr_line (start 135 115) (end 133 113) (angle 90) (layer Edge.Cuts) (width 0.1))
   (gr_text mosi (at 148.5 122.5) (layer F.Cu)
     (effects (font (size 1.2 1.2) (thickness 0.3)))
@@
     (effects (font (size 1.2 1.2) (thickness 0.3)))
   )
-  (gr_text "18, 19, \ngnd" (at 139 137) (layer F.Cu)
+  (gr_text "18, 19, \ngnd" (at 138.5 136.75) (layer F.Cu)
     (effects (font (size 1.2 1.2) (thickness 0.3)))
   )
-  (gr_text 9 (at 136 133) (layer F.Cu)
+  (gr_text 9 (at 149.25 133) (layer F.Cu)
     (effects (font (size 1.5 1.5) (thickness 0.3)))
   )
-  (gr_text 8 (at 136 129) (layer F.Cu)
+  (gr_text 8 (at 149.25 129) (layer F.Cu)
     (effects (font (size 1.5 1.5) (thickness 0.3)))
   )
-  (gr_text 2 (at 136 125) (layer F.Cu)
+  (gr_text 2 (at 149.25 125) (layer F.Cu)
     (effects (font (size 1.5 1.5) (thickness 0.3)))
   )
@@
   (gr_line (start 151 115) (end 151 141) (angle 90) (layer Edge.Cuts) (width 0.1))
   (gr_line (start 135 115) (end 151 115) (angle 90) (layer Edge.Cuts) (width 0.1))
-  (gr_line (start 135 141) (end 135 115) (angle 90) (layer Edge.Cuts) (width 0.1))
-  (segment (start 143.45 125) (end 143.45 119.45) (width 0.4) (layer F.Cu) (net 1) (status 800000))
-  (segment (start 143.45 119.45) (end 143 119) (width 0.4) (layer F.Cu) (net 1) (status C00000))
+  (segment (start 143.45 125) (end 143.45 119.45) (width 0.4) (layer F.Cu) (net 1))
+  (segment (start 143.45 119.45) (end 143 119) (width 0.4) (layer F.Cu) (net 1))
   (segment (start 141.9525 125) (end 143.45 125) (width 0.4) (layer F.Cu) (net 1))
   (segment (start 143.45 125) (end 145.0475 125) (width 0.4) (layer F.Cu) (net 1))
@@
   (segment (start 143.55 133) (end 145.0475 133) (width 0.4) (layer F.Cu) (net 2))
   (segment (start 143.55 129) (end 143.55 127.7) (width 0.4) (layer F.Cu) (net 3))
-  (segment (start 146 120.9) (end 147.95 118.95) (width 0.4) (layer F.Cu) (net 3) (status 800000))
+  (segment (start 146 120.9) (end 147.95 118.95) (width 0.4) (layer F.Cu) (net 3))
   (segment (start 146 126.5) (end 146 120.9) (width 0.4) (layer F.Cu) (net 3))
   (segment (start 145.7 126.8) (end 146 126.5) (width 0.4) (layer F.Cu) (net 3))
@@
   (segment (start 141.9525 129) (end 143.55 129) (width 0.4) (layer F.Cu) (net 3))
   (segment (start 143.55 129) (end 145.0475 129) (width 0.4) (layer F.Cu) (net 3))
+  (segment (start 137 125) (end 136.25 125) (width 0.4) (layer F.Cu) (net 4))
   (segment (start 140.0475 125) (end 137 125) (width 0.4) (layer F.Cu) (net 4))
+  (segment (start 133.284 115.034) (end 129.417 115.034) (width 0.4) (layer F.Cu) (net 4) (status 800000))
+  (segment (start 134.75 116.5) (end 133.284 115.034) (width 0.4) (layer F.Cu) (net 4))
+  (segment (start 134.75 123.5) (end 134.75 116.5) (width 0.4) (layer F.Cu) (net 4))
+  (segment (start 136.25 125) (end 134.75 123.5) (width 0.4) (layer F.Cu) (net 4))
+  (segment (start 137 129) (end 136 129) (width 0.4) (layer F.Cu) (net 5))
   (segment (start 140.0475 129) (end 137 129) (width 0.4) (layer F.Cu) (net 5))
+  (segment (start 133.456 131.544) (end 129.417 131.544) (width 0.4) (layer F.Cu) (net 5) (status 800000))
+  (segment (start 136 129) (end 133.456 131.544) (width 0.4) (layer F.Cu) (net 5))
+  (segment (start 137 133) (end 135 133) (width 0.4) (layer F.Cu) (net 6))
   (segment (start 140.0475 133) (end 137 133) (width 0.4) (layer F.Cu) (net 6))
+  (segment (start 133.662 134.338) (end 129.417 134.338) (width 0.4) (layer F.Cu) (net 6) (status 800000))
+  (segment (start 135 133) (end 133.662 134.338) (width 0.4) (layer F.Cu) (net 6))
+  (segment (start 133.25 126) (end 133.25 126.25) (width 0.4) (layer B.Cu) (net 7))
+  (segment (start 132.02 127.48) (end 129.417 127.48) (width 0.4) (layer B.Cu) (net 7) (status 800000))
+  (segment (start 133.25 126.25) (end 132.02 127.48) (width 0.4) (layer B.Cu) (net 7))
+  (segment (start 133.25 126) (end 132 124.75) (width 0.4) (layer B.Cu) (net 7))
+  (segment (start 144 138) (end 144 129) (width 0.4) (layer B.Cu) (net 7) (status 400000))
+  (segment (start 144 129) (end 141 126) (width 0.4) (layer B.Cu) (net 7))
+  (segment (start 141 126) (end 133.25 126) (width 0.4) (layer B.Cu) (net 7))
   (segment (start 146.9525 133) (end 146.9525 135.0475) (width 0.4) (layer F.Cu) (net 7))
   (segment (start 146.9525 135.0475) (end 144 138) (width 0.4) (layer F.Cu) (net 7))
+  (via (at 144 138) (size 0.889) (layers F.Cu B.Cu) (net 7) (status C00000))
+  (segment (start 129.481 124.75) (end 129.417 124.686) (width 0.4) (layer B.Cu) (net 7) (status C00000))
+  (segment (start 132 124.75) (end 129.481 124.75) (width 0.4) (layer B.Cu) (net 7) (status 800000))
   (segment (start 146.9525 129) (end 146.9525 133) (width 0.4) (layer F.Cu) (net 7))
   (segment (start 146.9525 125) (end 146.9525 129) (width 0.4) (layer F.Cu) (net 7))
+  (zone (net 7) (net_name GND) (layer F.Cu) (hatch edge 0.508)
+    (connect_pads (clearance 0.508))
+    (min_thickness 0.254)
+    (fill (arc_segments 16) (thermal_gap 0.508) (thermal_bridge_width 0.508))
+    (polygon
+      (pts
+        (xy 151 141) (xy 135 141) (xy 133 143) (xy 133 146.25) (xy 132.5 146.75)
+        (xy 128 146.75) (xy 128 111) (xy 132.5 111) (xy 133 111.5) (xy 133 113)
+        (xy 135 115) (xy 151 115)
+      )
+    )
+  )
+  (zone (net 7) (net_name GND) (layer B.Cu) (hatch edge 0.508)
+    (connect_pads (clearance 0.508))
+    (min_thickness 0.254)
+    (fill (arc_segments 16) (thermal_gap 0.508) (thermal_bridge_width 0.508))
+    (polygon
+      (pts
+        (xy 151 141) (xy 135 141) (xy 133 143) (xy 133 146.25) (xy 132.5 146.75)
+        (xy 128 146.75) (xy 128 111) (xy 132.5 111) (xy 133 111.5) (xy 133 113)
+        (xy 135 115) (xy 151 115)
+      )
+    )
+  )
 )
