File: scheme/main/main.sch (KiCad schematic (older format))
At the start: 31 parts

Commit message: a
Parts:
- removed X?: 8MHz, symbol CRYSTAL
- added D1: LED, ~, symbol LED
- added K1: swd, symbol CONN_3
- added P3, P5: CONN_20X2_F, symbol CONN_20X2
- added P4, P7: CONN_20X2_M, symbol CONN_20X2
- added P6: +, ~, symbol TST
- added P8: -, ~, symbol TST
- added R1: 100, ~, symbol R
- added R5: 1k, symbol R
- added U1: CRYSTAL-4PIN, ~, symbol CRYSTAL-4PIN
- C5: renamed from C?; value 1u -> 10u
- gave numbers to parts that had none: 29
Connections:
- net labels added: pb10-scl2, pb11-sda2, pb6-scl1, pb7-sda1, pc14, pc15
- net labels removed: flash-mode, op-mode, pb1, pb10, pb11, pb2, pb6, pb7
- wire segments 129 -> 305
- no-connect marks 2 -> 4
Other:
- moved on the sheet: C1, C2, C3, C4, C5, C6, C7, C8, P1, P2, R2, R3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

Commit message: a
Parts:
- removed K2: swd, symbol CONN_3
Connections:
- wire segments 305 -> 301
Changed lines of the file:
@@
 Sheet 1 1
 Title ""
-Date "14 nov 2014"
+Date "15 nov 2014"
 Rev "0.1"
 Comp ""
@@
 	1    0    0    -1
 $EndComp
-Wire Wire Line
-	16150 1500 17200 1500
-Wire Wire Line
-	16150 1600 17200 1600
-Wire Wire Line
-	17200 1700 17150 1700
-Wire Wire Line
-	17150 1700 17150 1950
-Text Label 16150 1600 0    60   ~ 0
-swd-clk
-Text Label 16150 1500 0    60   ~ 0
-swd-io
-$Comp
-L GND #PWR012
-U 1 1 54645233
-P 17150 1950
-F 0 "#PWR012" H 17150 1950 30  0001 C CNN
-F 1 "GND" H 17150 1880 30  0001 C CNN
-F 2 "" H 17150 1950 60  0001 C CNN
-F 3 "" H 17150 1950 60  0001 C CNN
-	1    17150 1950
-	1    0    0    -1
-$EndComp
-$Comp
-L CONN_3 K2
-U 1 1 54645239
-P 17550 1600
-F 0 "K2" V 17500 1600 50  0000 C CNN
-F 1 "swd" V 17600 1600 40  0000 C CNN
-F 2 "" H 17550 1600 60  0001 C CNN
-F 3 "" H 17550 1600 60  0001 C CNN
-	1    17550 1600
-	1    0    0    -1
-$EndComp

Commit message: a
Other:
- moved on the sheet: D1, R5

Commit message: a
Parts:
- removed U3: MICRO-USB-B, ~, symbol MICRO-USB-B
- added U?: MICRO-USB-B, ~, symbol MICRO-USB-B
Connections:
- wire segments 301 -> 304
Changed lines of the file:
@@
 Sheet 1 1
 Title ""
-Date "15 nov 2014"
+Date "16 nov 2014"
 Rev "0.1"
 Comp ""
@@
 	19050 3050 19050 3200
 Wire Wire Line
-	20100 2500 20300 2500
-Wire Wire Line
 	20300 2300 20100 2300
 Wire Wire Line
 	20100 2300 20100 3000
-Connection ~ 20100 2500
 Wire Wire Line
 	20300 2100 19050 2100
@@
 F 3 "" H 19050 2800 60  0001 C CNN
 	1    19050 2800
-	1    0    0    -1
-$EndComp
-$Comp
-L MICRO-USB-B U3
-U 1 1 546452F2
-P 21200 2000
-F 0 "U3" H 21200 1600 60  0000 C CNN
-F 1 "MICRO-USB-B" H 21200 2400 60  0000 C CNN
-F 2 "~" H 21200 2000 60  0000 C CNN
-F 3 "~" H 21200 2000 60  0000 C CNN
-	1    21200 2000
 	1    0    0    -1
 $EndComp
@@
 Wire Wire Line
 	11500 7950 11400 7950
+$Comp
+L MICRO-USB-B U?
+U 1 1 54685272
+P 20850 1900
+F 0 "U?" H 20850 1950 60  0000 C CNN
+F 1 "MICRO-USB-B" H 20850 1750 60  0000 C CNN
+F 2 "~" H 20850 1900 60  0000 C CNN
+F 3 "~" H 20850 1900 60  0000 C CNN
+	1    20850 1900
+	0    -1   -1   0
+$EndComp
+Wire Wire Line
+	20750 2700 20750 2800
+Wire Wire Line
+	20950 2700 20950 2800
+Wire Wire Line
+	20750 1100 20750 1000
+Wire Wire Line
+	20950 1100 20950 1000
+$Comp
+L GND #PWR?
+U 1 1 546857A5
+P 20750 1000
+F 0 "#PWR?" H 20750 1000 30  0001 C CNN
+F 1 "GND" H 20750 930 30  0001 C CNN
+F 2 "" H 20750 1000 60  0001 C CNN
+F 3 "" H 20750 1000 60  0001 C CNN
+	1    20750 1000
+	-1   0    0    1
+$EndComp
+$Comp
+L GND #PWR?
+U 1 1 546857AB
+P 20950 1000
+F 0 "#PWR?" H 20950 1000 30  0001 C CNN
+F 1 "GND" H 20950 930 30  0001 C CNN
+F 2 "" H 20950 1000 60  0001 C CNN
+F 3 "" H 20950 1000 60  0001 C CNN
+	1    20950 1000
+	-1   0    0    1
+$EndComp
+$Comp
+L GND #PWR?
+U 1 1 546857B1
+P 20950 2800
+F 0 "#PWR?" H 20950 2800 30  0001 C CNN
+F 1 "GND" H 20950 2730 30  0001 C CNN
+F 2 "" H 20950 2800 60  0001 C CNN
+F 3 "" H 20950 2800 60  0001 C CNN
+	1    20950 2800
+	1    0    0    -1
+$EndComp
+$Comp
+L GND #PWR?
+U 1 1 546857B7
+P 20750 2800
+F 0 "#PWR?" H 20750 2800 30  0001 C CNN
+F 1 "GND" H 20750 2730 30  0001 C CNN
+F 2 "" H 20750 2800 60  0001 C CNN
+F 3 "" H 20750 2800 60  0001 C CNN
+	1    20750 2800
+	1    0    0    -1
+$EndComp
 $EndSCHEMATC

Commit message: a
Parts:
- gave numbers to parts that had none: 1
Connections:
- wire segments 304 -> 308
- no-connect marks 4 -> 2
Changed lines of the file:
@@
 Sheet 1 1
 Title ""
-Date "16 nov 2014"
+Date "17 nov 2014"
 Rev "0.1"
 Comp ""
@@
 	3150 6400 3150 5800
 Connection ~ 2700 6400
-NoConn ~ 2700 4800
-NoConn ~ 2300 6200
 $Comp
 L R R1
@@
 	11500 7950 11400 7950
 $Comp
-L MICRO-USB-B U?
+L MICRO-USB-B U3
 U 1 1 54685272
 P 20850 1900
-F 0 "U?" H 20850 1950 60  0000 C CNN
+F 0 "U3" H 20850 1950 60  0000 C CNN
 F 1 "MICRO-USB-B" H 20850 1750 60  0000 C CNN
 F 2 "~" H 20850 1900 60  0000 C CNN
@@
 	20950 1100 20950 1000
 $Comp
-L GND #PWR?
+L GND #PWR063
 U 1 1 546857A5
 P 20750 1000
-F 0 "#PWR?" H 20750 1000 30  0001 C CNN
+F 0 "#PWR063" H 20750 1000 30  0001 C CNN
 F 1 "GND" H 20750 930 30  0001 C CNN
 F 2 "" H 20750 1000 60  0001 C CNN
@@
 $EndComp
 $Comp
-L GND #PWR?
+L GND #PWR064
 U 1 1 546857AB
 P 20950 1000
-F 0 "#PWR?" H 20950 1000 30  0001 C CNN
+F 0 "#PWR064" H 20950 1000 30  0001 C CNN
 F 1 "GND" H 20950 930 30  0001 C CNN
 F 2 "" H 20950 1000 60  0001 C CNN
@@
 $EndComp
 $Comp
-L GND #PWR?
+L GND #PWR065
 U 1 1 546857B1
 P 20950 2800
-F 0 "#PWR?" H 20950 2800 30  0001 C CNN
+F 0 "#PWR065" H 20950 2800 30  0001 C CNN
 F 1 "GND" H 20950 2730 30  0001 C CNN
 F 2 "" H 20950 2800 60  0001 C CNN
@@
 $EndComp
 $Comp
-L GND #PWR?
+L GND #PWR066
 U 1 1 546857B7
 P 20750 2800
-F 0 "#PWR?" H 20750 2800 30  0001 C CNN
+F 0 "#PWR066" H 20750 2800 30  0001 C CNN
 F 1 "GND" H 20750 2730 30  0001 C CNN
 F 2 "" H 20750 2800 60  0001 C CNN
@@
 	1    0    0    -1
 $EndComp
+Wire Wire Line
+	2700 4800 2700 4750
+Wire Wire Line
+	2700 4750 2900 4750
+Wire Wire Line
+	2900 4750 2900 4850
+$Comp
+L GND #PWR067
+U 1 1 54697E25
+P 2900 4850
+F 0 "#PWR067" H 2900 4850 30  0001 C CNN
+F 1 "GND" H 2900 4780 30  0001 C CNN
+F 2 "" H 2900 4850 60  0001 C CNN
+F 3 "" H 2900 4850 60  0001 C CNN
+	1    2900 4850
+	1    0    0    -1
+$EndComp
+Wire Wire Line
+	2300 6200 2300 6300
+$Comp
+L GND #PWR068
+U 1 1 54697F7A
+P 2300 6300
+F 0 "#PWR068" H 2300 6300 30  0001 C CNN
+F 1 "GND" H 2300 6230 30  0001 C CNN
+F 2 "" H 2300 6300 60  0001 C CNN
+F 3 "" H 2300 6300 60  0001 C CNN
+	1    2300 6300
+	1    0    0    -1
+$EndComp

Commit message: a
Changed lines of the file:
@@
 Sheet 1 1
 Title ""
-Date "17 nov 2014"
+Date "19 nov 2014"
 Rev "0.1"
 Comp ""
@@
 F 3 "~" H 20850 1900 60  0000 C CNN
 	1    20850 1900
-	0    -1   -1   0
-$EndComp
-Wire Wire Line
+	0    -1   1    0
+$EndComp
+Wire Wire Line
