File: scheme/main/main.kicad_pcb (KiCad board)
At the start: 2 copper layers, 39 parts, among them J1 USB_A, K1 swd, P1 mode, P2 rst, P3 CONN_20X2_F, P4 CONN_20X2_M, P5 CONN_20X2_F, P6 +, P7 CONN_20X2_M, P8 -, U1 CRYSTAL-4PIN, U2 MCP1703T-3302E/CB

Commit message: a
Parts:
- moved R5 125.9 mm to (92.2, 88.8)
- moved R2 124.9 mm to (116.0, 63.0), turned to 90 degrees
- moved P1 40.7 mm to (113.5, 62.8), turned to 270 degrees
Changed lines of the file:
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@@
   )
   (module SM0805 (layer F.Cu)
-    (at 12 -6.25)
-    (attr smd)
-    (fp_text reference R2 (at 0 -0.3175) (layer F.SilkS)
-      (effects (font (size 0.50038 0.50038) (thickness 0.10922)))
-    )
-    (fp_text value 10k (at 0 0.381) (layer F.SilkS)
-      (effects (font (size 0.50038 0.50038) (thickness 0.10922)))
-    )
-    (fp_circle (center -1.651 0.762) (end -1.651 0.635) (layer F.SilkS) (width 0.09906))
-    (fp_line (start -0.508 0.762) (end -1.524 0.762) (layer F.SilkS) (width 0.09906))
-    (fp_line (start -1.524 0.762) (end -1.524 -0.762) (layer F.SilkS) (width 0.09906))
-    (fp_line (start -1.524 -0.762) (end -0.508 -0.762) (layer F.SilkS) (width 0.09906))
-    (fp_line (start 0.508 -0.762) (end 1.524 -0.762) (layer F.SilkS) (width 0.09906))
-    (fp_line (start 1.524 -0.762) (end 1.524 0.762) (layer F.SilkS) (width 0.09906))
-    (fp_line (start 1.524 0.762) (end 0.508 0.762) (layer F.SilkS) (width 0.09906))
-    (pad 1 smd rect (at -0.9525 0) (size 0.889 1.397)
+    (at 116 63 90)
+    (attr smd)
+    (fp_text reference R2 (at 0 -0.3175 90) (layer F.SilkS)
+      (effects (font (size 0.50038 0.50038) (thickness 0.10922)))
+    )
+    (fp_text value 10k (at 0 0.381 90) (layer F.SilkS)
+      (effects (font (size 0.50038 0.50038) (thickness 0.10922)))
+    )
+    (fp_circle (center -1.651 0.762) (end -1.651 0.635) (layer F.SilkS) (width 0.09906))
+    (fp_line (start -0.508 0.762) (end -1.524 0.762) (layer F.SilkS) (width 0.09906))
+    (fp_line (start -1.524 0.762) (end -1.524 -0.762) (layer F.SilkS) (width 0.09906))
+    (fp_line (start -1.524 -0.762) (end -0.508 -0.762) (layer F.SilkS) (width 0.09906))
+    (fp_line (start 0.508 -0.762) (end 1.524 -0.762) (layer F.SilkS) (width 0.09906))
+    (fp_line (start 1.524 -0.762) (end 1.524 0.762) (layer F.SilkS) (width 0.09906))
+    (fp_line (start 1.524 0.762) (end 0.508 0.762) (layer F.SilkS) (width 0.09906))
+    (pad 1 smd rect (at -0.9525 0 90) (size 0.889 1.397)
       (layers F.Cu F.Paste F.Mask)
       (net 47 N-0000052)
     )
-    (pad 2 smd rect (at 0.9525 0) (size 0.889 1.397)
+    (pad 2 smd rect (at 0.9525 0 90) (size 0.889 1.397)
       (layers F.Cu F.Paste F.Mask)
       (net 37 GND)
@@
   )
   (module SM0805 (layer F.Cu)
-    (at 12 -8.25)
+    (at 92.25 88.75)
     (attr smd)
     (fp_text reference R5 (at 0 -0.3175) (layer F.SilkS)
@@
   )
   (module PIN_ARRAY_2X1 (layer F.Cu)
-    (at 73 59.25)
+    (at 113.5 62.75 270)
     (descr "Connecteurs 2 pins")
     (tags "CONN DEV")
-    (fp_text reference P1 (at 0 -1.905) (layer F.SilkS)
+    (fp_text reference P1 (at 0 -1.905 270) (layer F.SilkS)
       (effects (font (size 0.762 0.762) (thickness 0.1524)))
     )
-    (fp_text value mode (at 0 -1.905) (layer F.SilkS) hide
+    (fp_text value mode (at 0 -1.905 270) (layer F.SilkS) hide
       (effects (font (size 0.762 0.762) (thickness 0.1524)))
     )
@@
     (fp_line (start 2.54 -1.27) (end 2.54 1.27) (layer F.SilkS) (width 0.1524))
     (fp_line (start 2.54 1.27) (end -2.54 1.27) (layer F.SilkS) (width 0.1524))
-    (pad 1 thru_hole rect (at -1.27 0) (size 1.524 1.524) (drill 1.016)
+    (pad 1 thru_hole rect (at -1.27 0 270) (size 1.524 1.524) (drill 1.016)
       (layers *.Cu *.Mask F.SilkS)
       (net 50 VDD)
     )
-    (pad 2 thru_hole circle (at 1.27 0) (size 1.524 1.524) (drill 1.016)
+    (pad 2 thru_hole circle (at 1.27 0 270) (size 1.524 1.524) (drill 1.016)
       (layers *.Cu *.Mask F.SilkS)
       (net 47 N-0000052)

Commit message: a
Parts:
- added U3: MICRO-USB-B, micro-usb-b, F.Cu at (196.0, 112.0)
- moved P6 250.8 mm to (206.0, 109.0)
- moved R13 229.4 mm to (193.0, 117.0), turned to 270 degrees
- moved P8 228.1 mm to (186.0, 109.0)
- moved R12 225.4 mm to (195.0, 117.0), turned to 90 degrees
- moved R11 225.4 mm to (197.0, 117.0), turned to 90 degrees
- moved R10 222.6 mm to (191.0, 117.0), turned to 270 degrees
- moved P7 153.2 mm to (230.0, 135.0), turned to 270 degrees
- moved P5 140.7 mm to (221.0, 135.0), turned to 270 degrees
- moved C1 94.6 mm to (179.0, 131.5)
- moved C2 94.6 mm to (181.5, 139.5)
- moved C4 94.6 mm to (176.5, 141.2)
- moved C6 94.6 mm to (188.8, 131.0)
- moved C7 94.6 mm to (198.5, 130.8)
- moved C8 94.6 mm to (198.8, 140.5)
- moved D1 94.6 mm to (165.0, 143.8)
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Connections:
- D1 pad 1: N-0000043 -> N-0000036
- D1 pad 2: N-0000050 (its old number) -> GND
- R5 pad 1: N-0000050 (its old number) -> N-0000044
- R5 pad 2: GND -> N-0000036
- stm1 pad 19: N-0000043 -> N-0000044
Other:
- board outline added: 50 x 60 mm

Commit message: a
Parts:
- moved P3 140.6 mm to (286.5, 140.0), turned to 0 degrees
- moved P4 130.5 mm to (286.5, 132.0), turned to 0 degrees
- moved P2 89.9 mm to (188.4, 56.6)
- moved K1 85.5 mm to (221.0, 45.0), turned to 90 degrees
- moved C1 83.3 mm to (193.3, 49.4), turned to 180 degrees
- moved C4 82.9 mm to (188.5, 59.2)
- moved C6 82.9 mm to (200.8, 49.0)
- moved C7 82.9 mm to (210.5, 48.8)
- moved C8 82.9 mm to (210.8, 58.5)
- moved R1 82.9 mm to (198.0, 53.5)
- moved R3 82.9 mm to (188.5, 61.2)
- moved U1 82.9 mm to (193.2, 53.5)
- moved stm1 82.9 mm to (205.8, 53.8)
- moved C2 82.8 mm to (193.3, 57.5)
- moved P5 81.5 mm to (286.5, 86.5), turned to 0 degrees
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Connections:
- R10 pad 1: N-0000040 -> N-0000036
- U1 pad 2: (no net) -> GND
- U1 pad 4: (no net) -> GND
- U3 pad 1: /Vusb -> GND
- U3 pad 2: N-0000041 -> N-0000036
- U3 pad 4: N-0000040 -> N-0000041
- U3 pad 5: GND -> /Vusb
- U3 pad 6: (no net) -> GND
- U3 pad 7: (no net) -> GND
- U3 pad 8: (no net) -> GND
- U3 pad 9: (no net) -> GND
Routing:
- net GND: track 0.00 -> 55.4 mm
- net N-0000046: track 0.00 -> 20.3 mm
- net /swd-clk: track 0.00 -> 16.5 mm
- net N-0000051: track 0.00 -> 13.6 mm
- net /swd-io: track 0.00 -> 13.0 mm
- net VDD: track 0.00 -> 8.53 mm
- net N-0000050: track 0.00 -> 5.63 mm
- net /usb-d+: track 0.00 -> 5.53 mm
- net /usb-d-: track 0.00 -> 5.41 mm
- net N-0000045: track 0.00 -> 2.70 mm
Other:
- net class Default: clearance 0.254 -> 0.24
- rule trace_clearance: 0.254 -> 0.24

Commit message: a
Parts:
- moved C5 305.1 mm to (277.5, 115.3), turned to 90 degrees
- moved C3 295.8 mm to (279.4, 113.1), turned to 90 degrees
- moved R4 291.2 mm to (275.5, 117.5), turned to 90 degrees
- moved R9 280.0 mm to (277.6, 93.5), turned to 90 degrees
- moved R6 269.3 mm to (264.9, 93.5), turned to 90 degrees
- moved J1 136.6 mm to (320.9, 97.7), turned to 0 degrees
- moved P8 124.1 mm to (309.6, 98.1)
- moved R10 112.9 mm to (303.4, 106.5), turned to 90 degrees
- moved R13 112.6 mm to (305.6, 115.3), turned to 180 degrees
- moved U3 109.5 mm to (305.5, 108.7), turned to 90 degrees
- moved P6 104.1 mm to (309.6, 119.6)
- moved D1 102.9 mm to (264.4, 117.0), turned to 90 degrees
- moved R5 98.9 mm to (265.4, 120.6), turned to 180 degrees
- moved R11 98.4 mm to (296.5, 110.1)
- moved R12 98.4 mm to (296.5, 108.3)
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Connections:
- U3 pad 1: GND -> /Vusb
- U3 pad 2: N-0000036 -> N-0000041
- U3 pad 4: N-0000041 -> N-0000036
- U3 pad 5: /Vusb -> GND
Routing:
- net N-0000041: track 0.00 -> 8.36 mm
- net N-0000042: track 0.00 -> 8.21 mm
- net GND: track 55.4 -> 49.4 mm
- net /swd-io: track 13.0 -> 7.46 mm
- net /swd-clk: track 16.5 -> 12.1 mm
- net /usb-d-: track 5.41 -> 6.01 mm

Commit message: a
Parts:
- D2, D3: footprint DO-214AB -> SOD323-W
- moved R8 286.5 mm to (275.1, 93.5), turned to 90 degrees
- moved R7 281.1 mm to (267.4, 93.5), turned to 90 degrees
- moved D2 259.7 mm to (304.6, 122.2), turned to 90 degrees
- moved D3 257.1 mm to (302.5, 115.2), turned to 270 degrees
- moved U2 252.8 mm to (301.4, 120.4), turned to 270 degrees
- moved C9 252.7 mm to (298.2, 116.4), turned to 0 degrees
- moved C10 249.3 mm to (298.5, 120.3), turned to 90 degrees
- moved J1 65.4 mm to (256.9, 111.1), turned to 180 degrees
- moved C3 0.40 mm to (279.0, 113.1)
- moved C5 0.30 mm to (277.2, 115.3)
- moved R4 0.20 mm to (275.3, 117.5)
Routing:
- net N-0000052: track 0.00 -> 4.54 mm
- net /pa0: track 0.00 -> 3.79 mm
- net /pa1: track 0.00 -> 3.79 mm
- net GND: track 49.4 -> 53.0 mm
- net /pa2: track 0.00 -> 2.19 mm
