File: scheme/usb-to-serial/usb-to-serial.sch (KiCad schematic (older format))
At the start: 36 parts, among them P1 CONN_6X2, Q1 MOS_P, U1 FT232BL, U2 LP5951MF-3.3, U3 MINI-USB-B, X1 CRYSTAL

Commit message: Copied needed libraries.
Parts:
- X1: symbol CRYSTAL -> Crystal
Changed lines of the file:
@@
-EESchema Schematic File Version 2  date Sat 13 Apr 2013 11:18:08 PM MSK
+EESchema Schematic File Version 2
+LIBS:usb-to-serial-rescue
 LIBS:power
 LIBS:device
@@
 LIBS:memory
 LIBS:xilinx
-LIBS:special
 LIBS:microcontrollers
 LIBS:dsp
@@
 LIBS:contrib
 LIBS:valves
-LIBS:ft232bl
-LIBS:my_comps
-LIBS:lp5951mf-3
-LIBS:usb
-LIBS:usb-to-serial-cache
-EELAYER 27 0
+EELAYER 25 0
 EELAYER END
 $Descr A3 16535 11693
@@
 $EndComp
 $Comp
-L CRYSTAL X1
+L Crystal X1
 U 1 1 51687701
 P 5600 7100
