File: scheme/csr-spi-ftdi/csr-spi-ftdi.kicad_pcb (KiCad board)
At the start: 2 copper layers, 0 parts

Commit message: a
Parts:
- added C1: 0.1uF, Capacitors_SMD:C_0805, F.Cu at (154.2, 91.6)
- added C2: 0.1uF, Capacitors_SMD:C_0805, F.Cu at (143.4, 103.6)
- added C3: 4u7, Capacitors_SMD:C_0805, F.Cu at (132.4, 116.4)
- added C4: 4u7, Capacitors_SMD:C_0805, F.Cu at (148.5, 105.0)
- added D1: LED_READ, LEDs:LED-5MM, F.Cu at (151.6, 83.2)
- added D2: LED_WRITE, LEDs:LED-5MM, F.Cu at (142.6, 81.6)
- added D3: LED_PWR, LEDs:LED-5MM, F.Cu at (163.2, 83.0)
- added P1: USB_B, Connect:USB_B, F.Cu at (125.4, 93.4)
- added P2: CONN_02X07, Pin_Headers:Pin_Header_Angled_2x07, F.Cu at (167.8, 96.2)
- added R1: 220, Resistors_SMD:R_0805, F.Cu at (144.8, 100.0)
- added R10: 220, Resistors_SMD:R_0805, F.Cu at (145.4, 93.6)
- added R11: 1k, Resistors_SMD:R_0805, F.Cu at (155.2, 105.2)
- added R12: 220, Resistors_SMD:R_0805, F.Cu at (150.0, 94.6)
- added R13: 1k, Resistors_SMD:R_0805, F.Cu at (154.8, 109.0)
- added R14: 1k, Resistors_SMD:R_0805, F.Cu at (155.4, 101.8)
- added R15: 1k, Resistors_SMD:R_0805, F.Cu at (145.2, 109.4)
- added R2: 220, Resistors_SMD:R_0805, F.Cu at (152.4, 97.4)
- added R3: 220, Resistors_SMD:R_0805, F.Cu at (136.4, 108.0)
- added R4: 220, Resistors_SMD:R_0805, F.Cu at (132.6, 105.8)
- added R5: 220, Resistors_SMD:R_0805, F.Cu at (146.2, 91.4)
- added R6: 220, Resistors_SMD:R_0805, F.Cu at (128.8, 104.0)
- added R7: 220, Resistors_SMD:R_0805, F.Cu at (150.4, 108.8)
- added R8: 220, Resistors_SMD:R_0805, F.Cu at (139.4, 116.4)
- added R9: 220, Resistors_SMD:R_0805, F.Cu at (150.8, 101.6)
- added U1: FT232RL, Housings_SSOP:SSOP-28_5.3x10.2mm_Pitch0.65mm, F.Cu at (137.0, 95.0)
- added U2: MCP1703T-3302E/CB, TO_SOT_Packages_SMD:SOT-23_Handsoldering, F.Cu at (136.6, 102.4)

Commit message: a
Parts:
- removed R1, R10, R12, R2, R3, R4, R5, R6, R7, R8, R9: 220, Resistors_SMD:R_0805
- P1: moved to B.Cu
- R11: value 1k -> 10k
- moved R15 42.3 mm to (116.5, 78.3)
- moved D3 40.9 mm to (122.7, 77.2), turned to 180 degrees
- moved R11 39.8 mm to (125.9, 78.2), turned to 90 degrees
- moved R13 38.9 mm to (131.0, 78.2), turned to 90 degrees
- moved R14 35.4 mm to (129.1, 78.2), turned to 90 degrees
- moved C3 32.7 mm to (124.2, 84.7), turned to 180 degrees
- moved P2 26.9 mm to (148.8, 77.0)
- moved C2 24.8 mm to (134.5, 80.5), turned to 90 degrees
- moved C1 24.6 mm to (129.7, 93.7), turned to 180 degrees
- moved D1 21.9 mm to (133.1, 71.5), turned to 270 degrees
- moved D2 18.9 mm to (126.7, 71.5), turned to 270 degrees
- moved C4 15.2 mm to (137.7, 94.3), turned to 270 degrees
- moved U1 8.49 mm to (132.2, 88.0), turned to 270 degrees
- moved U2 8.41 mm to (134.3, 94.3)
- moved P1 6.80 mm to (125.2, 86.6)
Connections:
- R11 pad 1: Net-(R11-Pad1) -> /cbus3
- U1 pad 1: Net-(R1-Pad1) -> TX
- U1 pad 12: Net-(R10-Pad1) -> /cbus4
- U1 pad 13: Net-(R5-Pad1) -> /cbus2
- U1 pad 14: Net-(R11-Pad1) -> /cbus3
- U1 pad 2: Net-(R3-Pad1) -> CS#
- U1 pad 22: Net-(R9-Pad1) -> /cbus1
- U1 pad 23: Net-(R4-Pad1) -> /cbus0
- U1 pad 3: Net-(R2-Pad1) -> CLK
- U1 pad 5: Net-(R6-Pad1) -> RX
- U1 pad 6: Net-(R8-Pad1) -> MOSI
- U1 pad 9: Net-(R7-Pad1) -> MISO
Routing:
- net GND: track 0.00 -> 26.6 mm
- net VUSB: track 0.00 -> 24.4 mm
- net D+: track 0.00 -> 6.43 mm
- net D-: track 0.00 -> 5.07 mm
- net 3V3: track 0.00 -> 1.80 mm

Commit message: Finished debug PCB.
Parts:
- removed R11: 10k, Resistors_SMD:R_0805
- added P10: TST, Measurement_Points:Measurement_Point_Round-SMD-Pad_Small, F.Cu at (132.6, 77.5)
- added P11: TST, Measurement_Points:Measurement_Point_Round-SMD-Pad_Small, F.Cu at (144.1, 91.3)
- added P3: TST, Measurement_Points:Measurement_Point_Round-SMD-Pad_Small, F.Cu at (131.0, 78.3)
- added P4: TST, Measurement_Points:Measurement_Point_Round-SMD-Pad_Small, F.Cu at (144.1, 87.7)
- added P5: TST, Measurement_Points:Measurement_Point_Round-SMD-Pad_Small, F.Cu at (144.1, 89.5)
- added P6: TST, Measurement_Points:Measurement_Point_Round-SMD-Pad_Small, F.Cu at (122.0, 79.4)
- added P7: TST, Measurement_Points:Measurement_Point_Round-SMD-Pad_Small, F.Cu at (123.8, 79.4)
- added P8: TST, Measurement_Points:Measurement_Point_Round-SMD-Pad_Small, F.Cu at (141.8, 93.8)
- added P9: TST, Measurement_Points:Measurement_Point_Round-SMD-Pad_Small, F.Cu at (134.5, 78.0)
- added R1: 220, Resistors_SMD:R_0805, F.Cu at (141.6, 91.3)
- added R2: 220, Resistors_SMD:R_0805, F.Cu at (141.6, 87.7)
- added R3: 220, Resistors_SMD:R_0805, F.Cu at (141.6, 89.5)
- added R5: 220, Resistors_SMD:R_0805, F.Cu at (132.6, 80.6)
- added R7: 220, Resistors_SMD:R_0805, F.Cu at (129.4, 80.6)
- added R8: 220, Resistors_SMD:R_0805, F.Cu at (131.0, 80.6)
- P2: value CONN_02X07 -> TST; footprint Pin_Headers:Pin_Header_Angled_2x07 -> Measurement_Points:Measurement_Point_Round-SMD-Pad_Small
- moved P2 19.4 mm to (129.4, 77.5)
- moved D2 18.6 mm to (140.4, 84.0), turned to 0 degrees
- moved D1 9.90 mm to (139.9, 78.7), turned to 180 degrees
- moved D3 5.36 mm to (117.5, 78.8)
- moved R13 4.04 mm to (127.8, 80.6)
- moved R14 3.76 mm to (126.2, 80.7)
- moved R15 3.54 mm to (120.0, 78.9), turned to 90 degrees
Connections:
- U1 pad 1: TX -> Net-(R1-Pad1)
- U1 pad 12: /cbus4 -> (no net)
- U1 pad 13: /cbus2 -> (no net)
- U1 pad 14: /cbus3 -> (no net)
- U1 pad 2: CS# -> Net-(R3-Pad1)
- U1 pad 22: /cbus1 -> (no net)
- U1 pad 23: /cbus0 -> (no net)
- U1 pad 3: CLK -> Net-(R2-Pad1)
- U1 pad 5: RX -> Net-(R5-Pad1)
- U1 pad 6: MOSI -> Net-(R8-Pad1)
- U1 pad 9: MISO -> Net-(R7-Pad1)
Routing:
- net GND: track 26.6 -> 118.3 mm
- net 3V3: track 1.80 -> 52.1 mm
- net Net-(D2-Pad2): track 0.00 -> 26.9 mm
- net VUSB: track 24.4 -> 49.9 mm
- net Net-(D1-Pad2): track 0.00 -> 15.0 mm
- net Net-(R1-Pad1): track 0.00 -> 11.9 mm
- net Net-(R3-Pad1): track 0.00 -> 11.6 mm
- net Net-(R2-Pad1): track 0.00 -> 10.9 mm
- net Net-(D3-Pad2): track 0.00 -> 6.17 mm
- net LED_WR#: track 0.00 -> 6.01 mm
- net LED_RD#: track 0.00 -> 5.05 mm
- net Net-(R8-Pad1): track 0.00 -> 4.16 mm
- net D-: track 5.07 -> 9.07 mm
- net Net-(R7-Pad1): track 0.00 -> 3.97 mm
- net Net-(R5-Pad1): track 0.00 -> 3.38 mm
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- added copper zone on B.Cu, net GND
- added copper zone on F.Cu, net GND
Other:
- board outline added: 33 x 21.5 mm
